Commit message: CAD model files & fixed .urdf file

File: matlab/mycobot.urdf (robot description, URDF)
Before this commit: robot firefighter, 7 links, 6 joints
Joints:
- joint joint2_to_joint1: origin xyz=0 0 0.162 rpy=0 0 0 -> xyz=0 0 0.1739 rpy=0 0 0
- joint joint4_to_joint3: origin xyz=0.13635 0 0    rpy=0 0 0 -> xyz=0.135 0 0    rpy=0 0 0
- joint joint5_to_joint4: origin xyz=0.1205 0 0.082  rpy= 0 0 1.57080 -> xyz=0.120 0 0.08878  rpy= 0 0 1.57080
- joint joint6_to_joint5: origin xyz=0 -0.084 0 rpy=1.5708 0 0 -> xyz=0 -0.095 0 rpy=1.5708 0 0
- joint joint6output_to_joint6: origin xyz=0 0.06635 0 rpy=-1.5708 0 0 -> xyz=0 0.06550 0 rpy=-1.5708 0 0
